File: EagleCAD/PCB Design/ECE411_Project1.brd (EAGLE design)
At the start: 160 x 100 mm, 37 parts, among them J1 0473460001_USBMICRO, U1 ATS160SM-1, U2 MIC29310-5.0WU, U3 NCP5501DT50RKG, U4 DCJACK_2.1MM_PTH

Commit message: Add files via upload
connections made and test passed
Parts:
- moved TP_SRVOPWR 159.1 mm to (155.5, 27.5)
- moved TP_PWM1 142.0 mm to (129.5, 58.0), turned to 270 degrees
- moved TP_PWM2 139.9 mm to (124.5, 58.0), turned to 270 degrees
- moved BUTTON_PAD 129.8 mm to (27.8, 58.2), turned to 180 degrees
- moved J1 109.2 mm to (75.4, 4.08), turned to 90 degrees
- moved TP_LED1 91.0 mm to (70.0, 21.0), turned to 90 degrees
- moved TP_LED2 84.0 mm to (65.0, 21.0), turned to 90 degrees
- moved C2 77.2 mm to (108.4, 58.0)
- moved C3 77.2 mm to (102.0, 58.0)
- moved C4 77.2 mm to (95.7, 58.0)
- moved C5 77.2 mm to (114.0, 58.1)
- moved R4 73.7 mm to (83.2, 37.1)
- moved LED1 73.6 mm to (83.2, 26.7)
- moved LED2 73.6 mm to (83.2, 31.8)
- moved R3 73.6 mm to (83.2, 43.2)
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Routing:
- net GND: track 0.00 -> 517.9 mm, vias 0 -> 16
- net VCC: track 0.00 -> 263.4 mm, vias 0 -> 6
- net PWM2: track 0.00 -> 160.3 mm, vias 0 -> 5
- net D-USB: track 0.00 -> 111.5 mm
- net SERVO_PWR: track 0.00 -> 110.8 mm, vias 0 -> 2
- net PWM1: track 0.00 -> 106.0 mm, vias 0 -> 2
- net /RST: track 0.00 -> 102.3 mm, vias 0 -> 2
- net D+USB: track 0.00 -> 96.3 mm, vias 0 -> 2
- net UNREG_PWR: track 0.00 -> 85.9 mm, vias 0 -> 2
- net D+MCU: track 0.00 -> 78.2 mm, vias 0 -> 3
- net D-MCU: track 0.00 -> 76.4 mm, vias 0 -> 4
- net N$6: track 0.00 -> 65.5 mm, vias 0 -> 2
- net N$10: track 0.00 -> 60.2 mm
- net N$8: track 0.00 -> 53.7 mm, vias 0 -> 2
- net N$16: track 0.00 -> 52.1 mm, vias 0 -> 2
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Other:
- board size 160 x 100 mm -> 160 x 65.5 mm
